File: midi.kicad_sch (KiCad schematic)
At the start: 22 parts, among them CN1 MIDI Out 1, CN2 MIDI In 1, CN3 MIDI Out 2, CN4 MIDI In 2, J4 UART46, J5 UART5, U6 6N137S-TA1, U7 6N137S-TA1

Commit message: 1. Update README with info on my KiCAD component library. 2. Add Fiducial markers. 3. Add LCSC IDs for all parts in BOM.
Parts:
- CNxx1: LCSC (none) -> C136686
- CNxxx1: LCSC (none) -> C879743
- J4: LCSC (none) -> C5156676
- J5: DPFNOTES (none) -> 4P 2.54mm Single Row 1x4P Plugin,P=2.54mm Pin Headers ROHS; LCSC (none) -> C5116483
- R13, R14, R26, R27: DPFNOTES (none) -> 62.5mW Thick Film Resistors 50V ±1% ±200ppm/℃ 47Ω 0402 Chip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; LCSC (none) -> C25118
- R15, R28: DPFNOTES (none) -> 62.5mW Thick Film Resistors 50V ±100ppm/℃ ±1% 220Ω 0402 Chi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; LCSC (none) -> C25091
- R16, R29: DPFNOTES (none) -> 62.5mW Thick Film Resistors 50V ±100ppm/℃ ±1% 470Ω 0402 Chi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; LCSC (none) -> C25117
- U6, U7: LCSC (none) -> C92651
Changed lines of the file:
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@@
 			)
 		)
-		(property "LCSC" ""
+		(property "LCSC" "C136686"
 			(at 24.13 194.31 0)
 			(effects
@@
 		(property "LCSC Part" "C92651"
 			(at 78.74 124.46 0)
+			(effects
+				(font
+					(size 1.27 1.27)
+				)
+				(hide yes)
+			)
+		)
+		(property "LCSC" "C92651"
+			(at 78.74 104.14 0)
 			(effects
 				(font
@@
 			)
 		)
-		(property "Datasheet" "~"
+		(property "Datasheet" "https://www.lcsc.com/datasheet/lcsc_datasheet_2205311900_UNI-ROYAL-Uniroyal-Elec-0402WGF4700TCE_C25117.pdf"
 			(at 99.06 49.53 0)
 			(effects
@@
 			)
 		)
-		(property "LCSC" ""
+		(property "LCSC" "C25117"
 			(at 99.06 49.53 0)
 			(effects
@@
 			)
 		)
-		(property "DPFNOTES" ""
+		(property "DPFNOTES" "62.5mW Thick Film Resistors 50V ±100ppm/℃ ±1% 470Ω 0402 Chip Resistor - Surface Mount ROHS"
 			(at 99.06 49.53 0)
 			(effects
@@
 		(property "LCSC Part" "C92651"
 			(at 78.74 72.39 0)
+			(effects
+				(font
+					(size 1.27 1.27)
+				)
+				(hide yes)
+			)
+		)
+		(property "LCSC" "C92651"
+			(at 78.74 52.07 0)
 			(effects
 				(font
@@
 			)
 		)
-		(property "Datasheet" "~"
+		(property "Datasheet" "https://www.lcsc.com/datasheet/lcsc_datasheet_2205311900_UNI-ROYAL-Uniroyal-Elec-0402WGF470JTCE_C25118.pdf"
 			(at 46.99 86.36 0)
 			(effects
@@
 			)
 		)
-		(property "LCSC" ""
+		(property "LCSC" "C25118"
 			(at 46.99 86.36 0)
 			(effects
@@
 			)
 		)
-		(property "DPFNOTES" ""
+		(property "DPFNOTES" "62.5mW Thick Film Resistors 50V ±1% ±200ppm/℃ 47Ω 0402 Chip Resistor - Surface Mount ROHS"
 			(at 46.99 86.36 0)
 			(effects
@@
 			)
 		)
-		(property "Datasheet" "~"
+		(property "Datasheet" "https://www.lcsc.com/datasheet/lcsc_datasheet_2205311900_UNI-ROYAL-Uniroyal-Elec-0402WGF470JTCE_C25118.pdf"
 			(at 46.99 31.75 0)
 			(effects
@@
 			)
 		)
-		(property "LCSC" ""
+		(property "LCSC" "C25118"
 			(at 46.99 31.75 0)
 			(effects
@@
 			)
 		)
-		(property "DPFNOTES" ""
+		(property "DPFNOTES" "62.5mW Thick Film Resistors 50V ±1% ±200ppm/℃ 47Ω 0402 Chip Resistor - Surface Mount ROHS"
 			(at 46.99 31.75 0)
 			(effects
@@
 		)
 		(property "Description" "Pin Header male with pin space 2.54mm. Pin Count -8"
+			(at 209.55 44.45 0)
+			(effects
+				(font
+					(size 1.27 1.27)
+				)
+				(hide yes)
+			)
+		)
+		(property "LCSC" "C5156676"
 			(at 209.55 44.45 0)
 			(effects
@@
 			)
 		)
-		(property "LCSC" ""
+		(property "LCSC" "C879743"
 			(at 26.67 177.8 0)
 			(effects
@@
 			)
 		)
-		(property "Datasheet" "~"
+		(property "Datasheet" "https://www.lcsc.com/datasheet/lcsc_datasheet_2205311900_UNI-ROYAL-Uniroyal-Elec-0402WGF4700TCE_C25117.pdf"
 			(at 99.06 101.6 0)
 			(effects
@@
 			)
 		)
-		(property "LCSC" ""
+		(property "LCSC" "C25117"
 			(at 99.06 101.6 0)
 			(effects
@@
 			)
 		)
-		(property "DPFNOTES" ""
+		(property "DPFNOTES" "62.5mW Thick Film Resistors 50V ±100ppm/℃ ±1% 470Ω 0402 Chip Resistor - Surface Mount ROHS"
 			(at 99.06 101.6 0)
 			(effects
@@
 			)
 		)
-		(property "Datasheet" "~"
+		(property "Datasheet" "https://www.lcsc.com/datasheet/lcsc_datasheet_2205311900_UNI-ROYAL-Uniroyal-Elec-0402WGF2200TCE_C25091.pdf"
 			(at 49.53 48.26 0)
 			(effects
@@
 			)
 		)
-		(property "LCSC" ""
+		(property "LCSC" "C25091"
 			(at 49.53 48.26 0)
 			(effects
@@
 			)
 		)
-		(property "DPFNOTES" ""
+		(property "DPFNOTES" "62.5mW Thick Film Resistors 50V ±100ppm/℃ ±1% 220Ω 0402 Chip Resistor - Surface Mount ROHS"
 			(at 49.53 48.26 0)
 			(effects
@@
 			)
 		)
-		(property "Datasheet" ""
+		(property "Datasheet" "https://wmsc.lcsc.com/wmsc/upload/file/pdf/v2/lcsc/2207291800_ZHOURI-2-54-1-4_C5116483.pdf"
 			(at 209.55 67.31 0)
 			(effects
@@
 		)
 		(property "Description" "Pin Header male with pin space 2.54mm. Pin Count -4"
+			(at 209.55 77.47 0)
+			(effects
+				(font
+					(size 1.27 1.27)
+				)
+				(hide yes)
+			)
+		)
+		(property "DPFNOTES" "4P 2.54mm Single Row 1x4P Plugin,P=2.54mm Pin Headers ROHS"
+			(at 209.55 77.47 0)
+			(effects
+				(font
+					(size 1.27 1.27)
+				)
+				(hide yes)
+			)
+		)
+		(property "LCSC" "C5116483"
 			(at 209.55 77.47 0)
 			(effects
@@
 			)
 		)
-		(property "Datasheet" "~"
+		(property "Datasheet" "https://www.lcsc.com/datasheet/lcsc_datasheet_2205311900_UNI-ROYAL-Uniroyal-Elec-0402WGF470JTCE_C25118.pdf"
 			(at 46.99 83.82 0)
 			(effects
@@
 			)
 		)
-		(property "LCSC" ""
+		(property "LCSC" "C25118"
 			(at 46.99 83.82 0)
 			(effects
@@
 			)
 		)
-		(property "DPFNOTES" ""
+		(property "DPFNOTES" "62.5mW Thick Film Resistors 50V ±1% ±200ppm/℃ 47Ω 0402 Chip Resistor - Surface Mount ROHS"
 			(at 46.99 83.82 0)
 			(effects
@@
 			)
 		)
-		(property "Datasheet" "~"
+		(property "Datasheet" "https://www.lcsc.com/datasheet/lcsc_datasheet_2205311900_UNI-ROYAL-Uniroyal-Elec-0402WGF470JTCE_C25118.pdf"
 			(at 46.99 34.29 0)
 			(effects
@@
 			)
 		)
-		(property "LCSC" ""
+		(property "LCSC" "C25118"
 			(at 46.99 34.29 0)
 			(effects
@@
 			)
 		)
-		(property "DPFNOTES" ""
+		(property "DPFNOTES" "62.5mW Thick Film Resistors 50V ±1% ±200ppm/℃ 47Ω 0402 Chip Resistor - Surface Mount ROHS"
 			(at 46.99 34.29 0)
 			(effects
@@
 			)
 		)
-		(property "Datasheet" "~"
+		(property "Datasheet" "https://www.lcsc.com/datasheet/lcsc_datasheet_2205311900_UNI-ROYAL-Uniroyal-Elec-0402WGF2200TCE_C25091.pdf"
 			(at 49.53 100.33 0)
 			(effects
@@
 			)
 		)
-		(property "LCSC" ""
+		(property "LCSC" "C25091"
 			(at 49.53 100.33 0)
 			(effects
@@
 			)
 		)
-		(property "DPFNOTES" ""
+		(property "DPFNOTES" "62.5mW Thick Film Resistors 50V ±100ppm/℃ ±1% 220Ω 0402 Chip Resistor - Surface Mount ROHS"
 			(at 49.53 100.33 0)
 			(effects

Commit message: 1. Remove unused components on schematic. 2. Find other color LEDs in JLCPCB.
Parts:
- removed CNxx1: PJ-3210-4A, easyeda2kicad:AUDIO_TH_PJ-3210-4A, symbol easyeda2kicad:PJ-3210-4A
- removed CNxxx1: PJ-321A-4A, easyeda2kicad:AUDIO-SMD_PJ-321A-4A, symbol easyeda2kicad:PJ-321A-4A
Other:
- note removed: "Surface mount"
- note removed: "Through-hole"

Commit message: Reviewing every item in the BOM against LCSC database. Found several errors already. Part way done.
Parts:
- C20, C44: DPFNOTES (none) -> 50V 100nF X7R ±10% 0402 Multilayer Ceramic Capacitors MLCC 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; JLC Basic Part (none) -> Basic
- CN1, CN2, CN3, CN4: DPFNOTES In-stock 3.5mm TRS -> -20℃~+70℃ 3.5mm Headphone Jack 30V 500mA SMD Audio Connecto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; JLC Basic Part (none) -> Extended; Manu Part (none) -> PJ-321A-4A; Manufacturer (none) -> Korean Hroparts Elec
- D6, D7: JLC Basic Part (none) -> Basic; Manu Part (none) -> 1N4148W; Manufacturer (none) -> ST(Semtech)
- J4: DPFNOTES (none) -> 8P 2.54mm Double Row 2x4P Plugin,P=2.54mm Pin Headers ROHS; JLC Basic Part (none) -> Extended; Manu Part (none) -> PZ2.54-2*4; Manufacturer (none) -> ZHOURI
- J5: JLC Basic Part (none) -> Extended; Manu Part (none) -> 2.54-1*4; Manufacturer (none) -> ZHOURI
- R13, R14, R26, R27: JLC Basic Part (none) -> Extended; Manu Part (none) -> 0402WGF470JTCE; Manufacturer (none) -> UNI-ROYAL(Uniroyal Elec)
